Commit message: Spawn robot from URDF via launch file

File: src/vehicle_description/urdf/vehicle.urdf (robot description, URDF)
Before this commit: robot vehicle_blue, 4 links, 3 joints
Links:
- added link base_footprint
Joints:
- added joint base_footprint_joint: type fixed, parent base_footprint, child base_link, origin xyz=0 0 0.4 rpy=0 0 0
